Commit message: joint6-tool0 added

File: irb120_robotiq85/irb120_robotiq85_gazebo/urdf/irb120_robotiq85_macro.xacro (robot description, xacro)
@@ -10,3 +10,9 @@
 		<origin xyz="0 0 0" rpy="0 0 0" />
 	</xacro:robotiq_85_gripper>
+	<link name="joint_6" />
+	<joint name="joint6-tool0" type="fixed">
+	<parent link="tool0" />
+	<child link="joint_6" />
+	<origin xyz="0.0 0.0 0.0" rpy="0.0 0.0 0.0" />
+	</joint>
 </robot>

Commit message: pid constants missing

File: irb120_robotiq85/irb120_robotiq85_gazebo/urdf/irb120_robotiq85_macro.xacro (robot description, xacro)
@@ -14,5 +14,5 @@
 	<parent link="tool0" />
 	<child link="joint_6" />
-	<origin xyz="0.0 0.0 0.0" rpy="0.0 0.0 0.0" />
+	<origin xyz="0.0 0.0 0.0" rpy="0.0 0.0 0.0"/>
 	</joint>
 </robot>
